File: Sustainer.sch (KiCad schematic (older format))
At the start: 1 part, among them U1 4070

Commit message: Small changes to the Schematics for readability More docs Add abstract for Booster
Changed lines of the file:
@@
 $Descr A4 11693 8268
 encoding utf-8
-Sheet 1 8
+Sheet 1 7
 Title ""
 Date ""
@@
 Wire Wire Line
 	6650 3500 7300 3500
-$Sheet
-S 6550 1000 2400 1000
-U 5DFFF192
-F0 "Examples" 50
-F1 "examples.sch" 50
-$EndSheet
 $EndSCHEMATC
