File: examples.sch (KiCad schematic (older format))
At the start: 13 parts

Commit message: Small changes to the Schematics for readability More docs Add abstract for Booster
Parts:
- gave numbers to parts that had none: 13
Changed lines of the file:
@@
 $EndDescr
 $Comp
-L 4xxx:40106 U?
+L 4xxx:40106 U6
 U 1 1 5DFFF535
 P 1250 1500
-F 0 "U?" H 1250 1650 50  0000 C CNN
+F 0 "U6" H 1250 1650 50  0000 C CNN
 F 1 "40106" H 1250 1300 50  0000 C CNN
 F 2 "" H 1250 1500 50  0001 C CNN
@@
 $EndComp
 $Comp
-L power:GND #PWR?
+L power:GND #PWR0101
 U 1 1 5DFFFDFA
 P 850 2000
-F 0 "#PWR?" H 850 1750 50  0001 C CNN
+F 0 "#PWR0101" H 850 1750 50  0001 C CNN
 F 1 "GND" H 855 1827 50  0000 C CNN
 F 2 "" H 850 2000 50  0001 C CNN
@@
 out
 $Comp
-L Device:R_POT RV?
+L Device:R_POT RV14
 U 1 1 5E0009AC
 P 1100 1000
-F 0 "RV?" V 985 1000 50  0000 C CNN
+F 0 "RV14" V 985 1000 50  0000 C CNN
 F 1 "100k" V 1100 1000 50  0000 C CNN
 F 2 "" H 1100 1000 50  0001 C CNN
@@
 $EndComp
 $Comp
-L Device:R R?
+L Device:R R5
 U 1 1 5E003E3E
 P 1600 1000
-F 0 "R?" V 1700 1000 50  0000 C CNN
+F 0 "R5" V 1700 1000 50  0000 C CNN
 F 1 "10k" V 1600 1000 50  0000 C CNN
 F 2 "" V 1530 1000 50  0001 C CNN
@@
 Connection ~ 850  1500
 $Comp
-L Device:C C?
+L Device:C C25
 U 1 1 5E00F1C8
 P 850 1750
-F 0 "C?" H 650 1700 50  0000 L CNN
+F 0 "C25" H 650 1700 50  0000 L CNN
 F 1 "0.1u" H 965 1705 50  0000 L CNN
 F 2 "" H 888 1600 50  0001 C CNN
@@
 	850  1900 850  2000
 $Comp
-L 4xxx:40106 U?
+L 4xxx:40106 U8
 U 1 1 5E015A61
 P 5800 1500
-F 0 "U?" H 5800 1650 50  0000 C CNN
+F 0 "U8" H 5800 1650 50  0000 C CNN
 F 1 "40106" H 5800 1300 50  0000 C CNN
 F 2 "" H 5800 1500 50  0001 C CNN
@@
 $EndComp
 $Comp
-L power:GND #PWR?
+L power:GND #PWR0102
 U 1 1 5E015A6B
 P 5400 2000
-F 0 "#PWR?" H 5400 1750 50  0001 C CNN
+F 0 "#PWR0102" H 5400 1750 50  0001 C CNN
 F 1 "GND" H 5405 1827 50  0000 C CNN
 F 2 "" H 5400 2000 50  0001 C CNN
@@
 out
 $Comp
-L Device:R_POT RV?
+L Device:R_POT RV16
 U 1 1 5E015A7A
 P 5650 1000
-F 0 "RV?" V 5535 1000 50  0000 C CNN
+F 0 "RV16" V 5535 1000 50  0000 C CNN
 F 1 "100k" V 5650 1000 50  0000 C CNN
 F 2 "" H 5650 1000 50  0001 C CNN
@@
 $EndComp
 $Comp
-L Device:R R?
+L Device:R R12
 U 1 1 5E015A84
 P 6150 1000
-F 0 "R?" V 6250 1000 50  0000 C CNN
+F 0 "R12" V 6250 1000 50  0000 C CNN
 F 1 "10k" V 6150 1000 50  0000 C CNN
 F 2 "" V 6080 1000 50  0001 C CNN
@@
 Connection ~ 5400 1500
 $Comp
-L Device:C C?
+L Device:C C27
 U 1 1 5E015A9A
 P 5400 1750
-F 0 "C?" H 5200 1700 50  0000 L CNN
+F 0 "C27" H 5200 1700 50  0000 L CNN
 F 1 "0.1u" H 5515 1705 50  0000 L CNN
 F 2 "" H 5438 1600 50  0001 C CNN
@@
 	5400 1900 5400 2000
 $Comp
-L 4xxx:40106 U?
+L 4xxx:40106 U7
 U 1 1 5E018E60
 P 4300 1500
-F 0 "U?" H 4300 1650 50  0000 C CNN
+F 0 "U7" H 4300 1650 50  0000 C CNN
 F 1 "40106" H 4300 1300 50  0000 C CNN
 F 2 "" H 4300 1500 50  0001 C CNN
@@
 $EndComp
 $Comp
-L power:GND #PWR?
+L power:GND #PWR0103
 U 1 1 5E018E6A
 P 3900 2000
-F 0 "#PWR?" H 3900 1750 50  0001 C CNN
+F 0 "#PWR0103" H 3900 1750 50  0001 C CNN
 F 1 "GND" H 3905 1827 50  0000 C CNN
 F 2 "" H 3900 2000 50  0001 C CNN
@@
 Connection ~ 4900 1500
 $Comp
-L Device:R_POT RV?
+L Device:R_POT RV15
 U 1 1 5E018E79
 P 4150 1000
-F 0 "RV?" V 4035 1000 50  0000 C CNN
+F 0 "RV15" V 4035 1000 50  0000 C CNN
 F 1 "100k" V 4150 1000 50  0000 C CNN
 F 2 "" H 4150 1000 50  0001 C CNN
@@
 $EndComp
 $Comp
-L Device:R R?
+L Device:R R10
 U 1 1 5E018E83
 P 4650 1000
-F 0 "R?" V 4750 1000 50  0000 C CNN
+F 0 "R10" V 4750 1000 50  0000 C CNN
 F 1 "10k" V 4650 1000 50  0000 C CNN
 F 2 "" V 4580 1000 50  0001 C CNN
@@
 Connection ~ 3900 1500
 $Comp
-L Device:C C?
+L Device:C C26
 U 1 1 5E018E99
 P 3900 1750
-F 0 "C?" H 3700 1700 50  0000 L CNN
+F 0 "C26" H 3700 1700 50  0000 L CNN
 F 1 "1u" H 4015 1705 50  0000 L CNN
 F 2 "" H 3938 1600 50  0001 C CNN
@@
 Simple oscillator
 $Comp
-L Device:D D?
+L Device:D D2
 U 1 1 5E01EF75
 P 5150 1500
-F 0 "D?" H 5150 1400 50  0000 C CNN
+F 0 "D2" H 5150 1400 50  0000 C CNN
 F 1 "Signal diode" H 5150 1600 50  0000 C CNN
 F 2 "" H 5150 1500 50  0001 C CNN
