File: output.sch (KiCad schematic (older format))
At the start: 9 parts, among them U4 LM386

Commit message: Some suggestions for breadboard layout
Parts:
- added C9: 1u, symbol Device:C
Connections:
- net input: now also C9.2; no longer R8.2
- new net: C9.1, R8.2
Changed lines of the file:
@@
 Comment4 ""
 $EndDescr
-Text HLabel 2850 3350 0    50   Input ~ 0
+Text HLabel 2100 3350 0    50   Input ~ 0
 input
 $Comp
@@
 Wire Wire Line
 	3400 2900 3500 2900
+$Comp
+L Device:C C9
+U 1 1 5E5A0857
+P 2700 3350
+F 0 "C9" V 2550 3350 50  0000 C CNN
+F 1 "1u" V 2850 3350 50  0000 C CNN
+F 2 "" H 2738 3200 50  0001 C CNN
+F 3 "~" H 2700 3350 50  0001 C CNN
+	1    2700 3350
+	0    1    1    0
+$EndComp
+Wire Wire Line
+	2550 3350 2100 3350
 $EndSCHEMATC

Commit message: More docs and suggested breadboard layouts
Parts:
- C9: footprint (none) -> Capacitor_THT:C_Rect_L7.2mm_W7.2mm_P5.00mm_FKS2_FKP2_MKS2_MKP2
Changed lines of the file:
@@
 F 0 "C9" V 2550 3350 50  0000 C CNN
 F 1 "1u" V 2850 3350 50  0000 C CNN
-F 2 "" H 2738 3200 50  0001 C CNN
+F 2 "Capacitor_THT:C_Rect_L7.2mm_W7.2mm_P5.00mm_FKS2_FKP2_MKS2_MKP2" H 2738 3200 50  0001 C CNN
 F 3 "~" H 2700 3350 50  0001 C CNN
 	1    2700 3350
